Commit message: added ball_follower

File: robot_bringup/urdf/ur.urdf.xacro (robot description, xacro)
@@ -17,7 +17,7 @@
   <xacro:arg name="visual_params" default="$(find robot_bringup)/config/$(arg ur_type)/visual_parameters.yaml"/>
   <xacro:arg name="transmission_hw_interface" default=""/>
-  <xacro:arg name="safety_limits" default="false"/>
-  <xacro:arg name="safety_pos_margin" default="0.15"/>
-  <xacro:arg name="safety_k_position" default="20"/>
+  <xacro:arg name="safety_limits" default="False"/>
+  <xacro:arg name="safety_pos_margin" default="0.015"/>
+  <xacro:arg name="safety_k_position" default="20.0"/>
   <!--When using gazebo simulations absolute paths are necessary.-->
   <xacro:arg name="force_abs_paths" default="true" />
@@ -38,5 +38,5 @@
     force_abs_paths="$(arg force_abs_paths)"
     >
-    <origin xyz="0 0 0" rpy="0 0 0" />          <!-- position robot in the world -->
+    <origin xyz="0 0 2" rpy="0 0 0" />          <!-- position robot in the world -->
   </xacro:ur_robot>
   <ros2_control name="ur5" type="system">

Commit message: prep rpesentation

File: robot_bringup/urdf/ur.urdf.xacro (robot description, xacro)
@@ -20,4 +20,5 @@
   <xacro:arg name="safety_pos_margin" default="0.015"/>
   <xacro:arg name="safety_k_position" default="20.0"/>
+  <xacro:property name="PI" value="3.1415926535897931"/>
   <!--When using gazebo simulations absolute paths are necessary.-->
   <xacro:arg name="force_abs_paths" default="true" />
@@ -38,5 +39,5 @@
     force_abs_paths="$(arg force_abs_paths)"
     >
-    <origin xyz="0 0 2" rpy="0 0 0" />          <!-- position robot in the world -->
+    <origin xyz="0 0 2" rpy="0 0 ${PI}" />          <!-- position robot in the world -->
   </xacro:ur_robot>
   <ros2_control name="ur5" type="system">
@@ -93,4 +94,7 @@
       </joint>
   </ros2_control>
+  <disable_collisions link1="upper_arm_link" link2="wrist_1_link" reason="intentionally disabled" />
+  <disable_collisions link1="upper_arm_link" link2="wrist_2_link" reason="intentionally disabled" />
+  <disable_collisions link1="upper_arm_link" link2="wrist_3_link" reason="intentionally disabled" />
   <gazebo>
       <plugin filename="gz_ros2_control-system" name="gz_ros2_control::GazeboSimROS2ControlPlugin">
